File: FW16_EPD.kicad_pcb (KiCad board)
At the start: 2 copper layers, 67.8 x 131 mm, 67 parts, among them J1 Conn_01x02, J2 Framework Input Module Connec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, J3 FH34SRJ-24S-0.5SH, J4 FH34SRJ-6S-0.5SH, Q1 DMG3404L, Q2 SSM3J338R, U1 RP2040, U2 W25Q128JVP, U3 MCP9808_DFN, Y1 12.000 MHz ABM8-272-T3

Commit message: finishing touches
Parts:
- moved R7 0.05 mm to (152.5, 122.5)
- moved R8 0.05 mm to (152.5, 121.5)
Routing:
- net /I2C_SCL: track 18.1 -> 20.8 mm, vias 0 -> 2
- net /EPD_TOUCH_RST#: track 15.9 -> 15.2 mm
- net GND: track 33.4 -> 32.8 mm, vias 159 -> 89
- net /EPD_TOUCH_INT: track 15.9 -> 15.4 mm
Other:
- rule pad_to_mask_clearance: 0.05 -> 0.038
- rule solder_mask_min_width: 0.2 -> 0.1
- board text added: "(c) arthomnix 2024 2024-10-03 r1.0"
- board text removed: "(c) arthomnix 2024 2024-07-10 r1.0"
- board text removed: "FW16_EPD r1.0 2024-07-10 (c) arthomnix 2024"
